File: RFM98PW-433S2_breakout.kicad_sch (KiCad schematic)
At the start: 14 parts, among them J1 U.FL-R-SMT-1(10), J2 Conn_01x05_Male, J3 Conn_01x03_Male, J4 Conn_01x02_Male, J5 Conn_01x02_Male, J6 Conn_01x02_Male, U1 RFM98PW-433S2

Commit message: first run
Parts:
- removed C1, C2: 6p, Capacitor_SMD:C_0603_1608Metric_Pad1.08x0.95mm_HandSolder, symbol Device:C
- removed L1: 18n, Inductor_SMD:L_0603_1608Metric_Pad1.05x0.95mm_HandSolder, symbol Device:L
- removed R1: 1M, Resistor_SMD:R_0603_1608Metric_Pad0.98x0.95mm_HandSolder, symbol Device:R
Connections:
- net +3V3: now also J6.1 (Pin_1); no longer J6.2 (Pin_2)
- net +5V: now also J5.1 (Pin_1); no longer J5.2 (Pin_2)
- net GND: now also J5.2 (Pin_2), J6.2 (Pin_2); no longer J5.1 (Pin_1), J6.1 (Pin_1)
- net RFM_DIO0: now also J3.3 (Pin_3); no longer J3.1 (Pin_1)
- net RFM_DIO2: now also J3.1 (Pin_1); no longer J3.3 (Pin_3)
- net RFM_DIO3: now also J4.2 (Pin_2); no longer J4.1 (Pin_1)
- net RFM_DIO4: now also J4.1 (Pin_1); no longer J4.2 (Pin_2)
- net RFM_MISO: now also J2.1 (Pin_1); no longer J2.5 (Pin_5)
- net RFM_MOSI: now also J2.2 (Pin_2); no longer J2.4 (Pin_4)
- net RFM_NSS: now also J2.4 (Pin_4); no longer J2.2 (Pin_2)
- net RFM_RESET: now also J2.5 (Pin_5); no longer J2.1 (Pin_1)
- net at J1.2: now also U1.1 (ANT)
